File: eagle/psoc_project/untitled.brd (EAGLE design)
At the start: 50 x 50 mm, 9 parts

Commit message: tt
Parts:
- JP1: device pinhead:1X02/90 -> pinhead:1X02
- moved JP1 1.27 mm to (43.2, 24.1), turned to 90 degrees
Changed lines of the file:
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@@
 <?xml version="1.0" encoding="utf-8"?>
 <!DOCTYPE eagle SYSTEM "eagle.dtd">
-<eagle version="7.6.0">
+<eagle version="6.5.0">
 <drawing>
 <settings>
@@
 <layers>
 <layer number="1" name="Top" color="4" fill="1" visible="yes" active="yes"/>
+<layer number="2" name="Route2" color="1" fill="3" visible="no" active="no"/>
+<layer number="3" name="Route3" color="4" fill="3" visible="no" active="no"/>
+<layer number="4" name="Route4" color="1" fill="4" visible="no" active="no"/>
+<layer number="5" name="Route5" color="4" fill="4" visible="no" active="no"/>
+<layer number="6" name="Route6" color="1" fill="8" visible="no" active="no"/>
+<layer number="7" name="Route7" color="4" fill="8" visible="no" active="no"/>
+<layer number="8" name="Route8" color="1" fill="2" visible="no" active="no"/>
+<layer number="9" name="Route9" color="4" fill="2" visible="no" active="no"/>
+<layer number="10" name="Route10" color="1" fill="7" visible="no" active="no"/>
+<layer number="11" name="Route11" color="4" fill="7" visible="no" active="no"/>
+<layer number="12" name="Route12" color="1" fill="5" visible="no" active="no"/>
+<layer number="13" name="Route13" color="4" fill="5" visible="no" active="no"/>
+<layer number="14" name="Route14" color="1" fill="6" visible="no" active="no"/>
+<layer number="15" name="Route15" color="4" fill="6" visible="no" active="no"/>
 <layer number="16" name="Bottom" color="1" fill="1" visible="yes" active="yes"/>
 <layer number="17" name="Pads" color="2" fill="1" visible="yes" active="yes"/>
@@
 <pass name="Default">
 <param name="RoutingGrid" value="50mil"/>
-<param name="AutoGrid" value="1"/>
-<param name="Efforts" value="0"/>
-<param name="TopRouterVariant" value="1"/>
 <param name="tpViaShape" value="round"/>
-<param name="PrefDir.1" value="a"/>
+<param name="PrefDir.1" value="|"/>
 <param name="PrefDir.2" value="0"/>
 <param name="PrefDir.3" value="0"/>
@@
 <param name="PrefDir.14" value="0"/>
 <param name="PrefDir.15" value="0"/>
-<param name="PrefDir.16" value="a"/>
+<param name="PrefDir.16" value="-"/>
 <param name="cfVia" value="8"/>
 <param name="cfNonPref" value="5"/>
@@
 <element name="C14" library="rcl" package="C0603" value="100NF" x="29.21" y="31.75"/>
 <element name="C15" library="rcl" package="C0603" value="1UF" x="29.21" y="38.1"/>
-<element name="JP1" library="pinhead" package="1X02/90" value="" x="44.45" y="24.13"/>
+<element name="JP1" library="pinhead" package="1X02" value="" x="43.18" y="24.13" rot="R90"/>
 </elements>
 <signals>
@@
 <contactref element="C11" pad="1"/>
 <contactref element="JP1" pad="1"/>
-<wire x1="35.14" y1="21.59" x2="43.18" y2="20.32" width="0" layer="19" extent="1-1"/>
+<wire x1="35.14" y1="21.59" x2="43.18" y2="22.86" width="0" layer="19" extent="1-1"/>
 <wire x1="35.14" y1="26.67" x2="35.14" y2="21.59" width="0" layer="19" extent="1-1"/>
 <wire x1="27.15" y1="27.005" x2="35.14" y2="26.67" width="0" layer="19" extent="1-1"/>
@@
 <wire x1="28.36" y1="31.75" x2="28.36" y2="38.1" width="0" layer="19" extent="1-1"/>
 <wire x1="27.65" y1="27.005" x2="28.36" y2="31.75" width="0" layer="19" extent="1-1"/>
-<wire x1="45.72" y1="20.32" x2="27.65" y2="27.005" width="0" layer="19" extent="1-1"/>
+<wire x1="43.18" y1="25.4" x2="27.65" y2="27.005" width="0" layer="19" extent="1-1"/>
 </signal>
 </signals>
